Commit message: feat(slam): update run_map.sh, robot.launch.py, and URDF for Go2 4-legged SLAM and TF alignment

File: src/go2_robot/go2_description/urdf/go2_description.urdf (robot description, URDF)
Before this commit: robot go2_description, 30 links, 29 joints
Joints:
- joint camera_joint: origin xyz=0.05 0 0.04 rpy=0 0 0 -> xyz=0.05 0 0.08 rpy=0 0 0
